File: goodmorningmat/Alarm_clock.sch (EAGLE design)
At the start: 24 parts, among them IC1 INA129U, IC2 MCP23017SP, J1 LOAD_CELL1X03-PTH, J2 LOAD_CELL1X03-PTH, Q1 32.768kHz

Commit message: Update Schematic
Other:
- note added: "Carl J. Anderson"
- note added: "Freshman Engineering Design"
Changed lines of the file:
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@@
 <description>Alarm Clock schematic for freshman design</description>
 <plain>
+<text x="139.7" y="-2.54" size="1.778" layer="91">Carl J. Anderson</text>
+<text x="139.7" y="-5.08" size="1.778" layer="91">
+Freshman Engineering Design</text>
 </plain>
 <instances>
@@
 </schematic>
 </drawing>
+<compatibility>
+<note version="6.3" minversion="6.2.2" severity="warning">
+Since Version 6.2.2 text objects can contain more than one line,
+which will not be processed correctly with this version.
+</note>
+</compatibility>
 </eagle>

Commit message: Update Schematic some more
Parts:
- added JP2: (no value), SparkFun-Connectors:M05PTH
Connections:
- new net SQW: JP2.3, RTC.SQW
- net 5V: now also JP2.1
- net GND: now also JP2.2
- net SCL: now also JP2.4
- net SDA: now also JP2.5
Changed lines of the file:
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@@
 <part name="SUPPLY10" library="SparkFun-Aesthetics" deviceset="5V" device=""/>
 <part name="SUPPLY11" library="SparkFun-Aesthetics" deviceset="5V" device=""/>
+<part name="JP2" library="SparkFun-Connectors" deviceset="M05" device="PTH"/>
+<part name="GND14" library="SparkFun-Aesthetics" deviceset="GND" device=""/>
 </parts>
 <sheets>
@@
 <instance part="SUPPLY10" gate="G$1" x="58.42" y="68.58" rot="R270"/>
 <instance part="SUPPLY11" gate="G$1" x="58.42" y="60.96" rot="R270"/>
+<instance part="JP2" gate="G$1" x="63.5" y="17.78" rot="R180"/>
+<instance part="GND14" gate="1" x="53.34" y="2.54"/>
 </instances>
 <busses>
@@
 <pinref part="S1" gate="S" pin="3"/>
 </segment>
+<segment>
+<pinref part="JP2" gate="G$1" pin="2"/>
+<wire x1="55.88" y1="20.32" x2="53.34" y2="20.32" width="0.1524" layer="91"/>
+<wire x1="53.34" y1="20.32" x2="53.34" y2="5.08" width="0.1524" layer="91"/>
+<pinref part="GND14" gate="1" pin="GND"/>
+</segment>
 </net>
 <net name="N$7" class="0">
@@
 <pinref part="RTC" gate="G$1" pin="VCC"/>
 <wire x1="43.18" y1="20.32" x2="48.26" y2="20.32" width="0.1524" layer="91"/>
-<wire x1="48.26" y1="20.32" x2="48.26" y2="27.94" width="0.1524" layer="91"/>
+<wire x1="48.26" y1="20.32" x2="48.26" y2="22.86" width="0.1524" layer="91"/>
 <pinref part="SUPPLY4" gate="G$1" pin="5V"/>
+<pinref part="JP2" gate="G$1" pin="1"/>
+<wire x1="48.26" y1="22.86" x2="48.26" y2="27.94" width="0.1524" layer="91"/>
+<wire x1="55.88" y1="22.86" x2="48.26" y2="22.86" width="0.1524" layer="91"/>
+<junction x="48.26" y="22.86"/>
 </segment>
 <segment>
@@
 <segment>
 <pinref part="RTC" gate="G$1" pin="SDA"/>
-<wire x1="43.18" y1="12.7" x2="48.26" y2="12.7" width="0.1524" layer="91"/>
 <label x="45.72" y="12.7" size="1.778" layer="95"/>
+<pinref part="JP2" gate="G$1" pin="5"/>
+<wire x1="55.88" y1="12.7" x2="43.18" y2="12.7" width="0.1524" layer="91"/>
 </segment>
 <segment>
@@
 <segment>
 <pinref part="RTC" gate="G$1" pin="SCL"/>
-<wire x1="43.18" y1="15.24" x2="48.26" y2="15.24" width="0.1524" layer="91"/>
 <label x="45.72" y="15.24" size="1.778" layer="95"/>
+<pinref part="JP2" gate="G$1" pin="4"/>
+<wire x1="55.88" y1="15.24" x2="43.18" y2="15.24" width="0.1524" layer="91"/>
 </segment>
 <segment>
@@
 </segment>
 </net>
+<net name="SQW" class="0">
+<segment>
+<pinref part="JP2" gate="G$1" pin="3"/>
+<pinref part="RTC" gate="G$1" pin="SQW"/>
+<wire x1="55.88" y1="17.78" x2="43.18" y2="17.78" width="0.1524" layer="91"/>
+<label x="45.72" y="17.78" size="1.778" layer="95"/>
+</segment>
+</net>
